File: A1200KB.sch (KiCad schematic (older format))
At the start: 97 parts, among them J1 Conn_01x32_Female, K1 ESC, K10 F9, K11 F10, K12 TILDE, K13 1, K14 2, K15 3, K16 4, K17 5, K18 6, K19 7, K2 F1, K20 8, K21 9, K22 0, K23 MINUS, K24 PLUS, K25 PIPE, K26 BS, K27 DEL, K28 HELP, K29 NUM_(, K3 F2, K30 NUM_), K31 NUM_DIV, K32 NUM_MULT, K33 TAB, K34 Q, K35 W, K36 E, K37 R, K38 T, K39 Y, K4 F3, K40 U, K41 I, K42 O, K43 P, K44 L.CURLY, K45 R.CURLY, K46 RETURN, K47 NUM_7, K48 NUM_8, K49 NUM_9, K5 F4, K50 NUM_MINUS, K51 CTRL, K52 CAPSLOCK, K53 A, K54 S, K55 D, K56 F, K57 G, K58 H, K59 J, K6 F5, K60 K, K61 L, K62 COLON, K63 \", K64 R.BLANK, K65 UP, K66 NUM_4, K67 NUM_5, K68 NUM_6, K69 NUM_PLUS, K7 F6, K70 L.SHIFT, K71 L.BLANK, K72 Z, K73 X, K74 C, K75 V, K76 B, K77 N, K78 M, K79 R.CROC, K8 F7, K80 L.CROC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

Commit message: Placed all
Parts:
- K28: footprint MX_Alps_Hybrid:MXOnly-1.25U-NoLED -> MX_Alps_Hybrid:MXOnly-1.5U-NoLED
Changed lines of the file:
@@
 EESchema Schematic File Version 4
+LIBS:A1200KB-cache
 EELAYER 29 0
 EELAYER END
@@
 F 0 "K28" H 17500 7039 60  0000 C CNN
 F 1 "HELP" H 17500 6933 60  0000 C CNN
-F 2 "MX_Alps_Hybrid:MXOnly-1.25U-NoLED" H 17500 6933 60  0001 C CNN
+F 2 "MX_Alps_Hybrid:MXOnly-1.5U-NoLED" H 17500 6933 60  0001 C CNN
 F 3 "" H 17500 6700 60  0000 C CNN
 	1    17500 6700

Commit message: Layout complete and art to ourpcb
Connections:
- net 3: now also K26.2 (ROW)
Changed lines of the file:
@@
 	6900 4800 7650 4800
 Wire Wire Line
-	7650 4800 7650 10100
+	7650 4800 7650 6200
 Connection ~ 7650 10100
 Wire Wire Line
@@
 Text Label 2200 5000 1    50   ~ 0
 31
+Wire Wire Line
+	15275 6875 15075 6875
+Wire Wire Line
+	15075 6875 15075 6200
+Wire Wire Line
+	15075 6200 7650 6200
+Connection ~ 7650 6200
+Wire Wire Line
+	7650 6200 7650 10100
 $EndSCHEMATC
