File: A1200KB.kicad_pcb (KiCad board)
At the start: 2 copper layers, 460 x 149 mm, 98 parts, among them J1 Conn_01x32_Female, K1 ESC, K10 F9, K11 F10, K12 TILDE, K13 1, K14 2, K15 3, K16 4, K17 5, K18 6, K19 7, K2 F1, K20 8, K21 9, K22 0, K23 MINUS, K24 PLUS, K25 PIPE, K26 BS, K27 DEL, K28 HELP, K29 NUM_(, K3 F2, K30 NUM_), K31 NUM_DIV, K32 NUM_MULT, K33 TAB, K34 Q, K35 W, K36 E, K37 R, K38 T, K39 Y, K4 F3, K40 U, K41 I, K42 O, K43 P, K44 L.CURLY, K45 R.CURLY, K46 RETURN, K47 NUM_7, K48 NUM_8, K49 NUM_9, K5 F4, K50 NUM_MINUS, K51 CTRL, K52 CAPSLOCK, K53 A, K54 S, K55 D, K56 F, K57 G, K58 H, K59 J, K6 F5, K60 K, K61 L, K62 COLON, K63 ", K64 R.BLANK, K65 UP, K66 NUM_4, K67 NUM_5, K68 NUM_6, K69 NUM_PLUS, K7 F6, K70 L.SHIFT, K71 L.BLANK, K72 Z, K73 X, K74 C, K75 V, K76 B, K77 N, K78 M, K79 R.CROC, K8 F7, K80 L.CROC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

Commit message: Placed all
Parts:
- removed REF**: 9U, MX_Alps_Hybrid:MX-9U-NoLED
- added IN CASE: 9U, MX_Alps_Hybrid:MX-9U-NoLED, F.Cu at (168.4, 138.7)
- K28: footprint MX_Alps_Hybrid:MXOnly-1.25U-NoLED -> MX_Alps_Hybrid:MXOnly-1.5U-NoLED
- moved K88 418.6 mm to (438.9, 119.9)
- moved K30 413.8 mm to (419.9, 62.8)
- moved K90 404.9 mm to (47.0, 138.7)
- moved K31 404.3 mm to (438.9, 62.8)
- moved K32 404.3 mm to (458.0, 62.8)
- moved K96 397.1 mm to (438.9, 139.0)
- moved K89 372.2 mm to (458.0, 129.6), turned to 90 degrees
- moved K48 364.4 mm to (419.9, 81.8)
- moved K47 364.4 mm to (400.8, 81.8)
- moved K49 364.4 mm to (438.9, 81.8)
- moved K50 364.4 mm to (458.0, 81.8)
- moved K91 362.4 mm to (70.9, 138.7)
- moved K12 348.1 mm to (35.7, 62.5)
- moved K75 302.5 mm to (140.5, 119.6)
- moved K76 290.9 mm to (159.5, 119.6)
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
Commit message: Layout complete and art to ourpcb
Parts:
- removed IN CASE: 9U, MX_Alps_Hybrid:MX-9U-NoLED
- moved K27 25.6 mm to (340.0, 62.5)
- moved K28 25.6 mm to (368.6, 62.5)
Connections:
- K26 pad 2: Net-(K26-Pad2) -> /3
Routing:
- net /16: track 0.00 -> 830.2 mm, vias 0 -> 1
- net /4: track 0.00 -> 685.8 mm
- net /3: track 0.00 -> 666.7 mm, vias 0 -> 1
- net /18: track 0.00 -> 605.4 mm, vias 0 -> 1
- net /15: track 0.00 -> 604.0 mm
- net /17: track 0.00 -> 561.4 mm, vias 0 -> 1
- net /19: track 0.00 -> 548.0 mm, vias 0 -> 1
- net /30: track 0.00 -> 543.0 mm
- net /24: track 0.00 -> 521.3 mm
- net /20: track 0.00 -> 507.9 mm, vias 0 -> 1
- net /2: track 0.00 -> 503.8 mm
- net /21: track 0.00 -> 502.7 mm, vias 0 -> 1
- net /22: track 0.00 -> 496.9 mm
- net /29: track 0.00 -> 491.2 mm
- net /27: track 0.00 -> 479.7 mm
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Other:
- rule trace_min: 0.2 -> 0.9
- board text added: "A1200KB"
- board text added: "Rev.1"
- board text added: "aeberbach"
- board text added: "grayunicorn.com"
- board text added: "march 2019"

Commit message: Routed again, cutout for LED PCB, sized for Al supports
Parts:
- added REF**: Banana_Jack_1Pin, Connector:Banana_Jack_1Pin, F.Cu at (213.3, 152.7)
- added REF**: Banana_Jack_1Pin, Connector:Banana_Jack_1Pin, F.Cu at (467.1, 152.0)
- added REF**: Banana_Jack_1Pin, Connector:Banana_Jack_1Pin, F.Cu at (65.6, 152.0)
- added REF**: Banana_Jack_1Pin, Connector:Banana_Jack_1Pin, F.Cu at (23.8, 151.9)
- added REF**: Banana_Jack_1Pin, Connector:Banana_Jack_1Pin, F.Cu at (16.8, 112.5)
- added REF**: Banana_Jack_1Pin, Connector:Banana_Jack_1Pin, F.Cu at (17.4, 52.4)
- added REF**: ALT-9U, MX_Alps_Hybrid:MX-9U, F.Cu at (164.4, 141.3)
- added REF**: Banana_Jack_1Pin, Connector:Banana_Jack_1Pin, F.Cu at (129.2, 18.2)
- added REF**: Banana_Jack_1Pin, Connector:Banana_Jack_1Pin, F.Cu at (53.4, 16.8)
- added REF**: Banana_Jack_1Pin, Connector:Banana_Jack_1Pin, F.Cu at (419.0, 19.3)
- added REF**: Banana_Jack_1Pin, Connector:Banana_Jack_1Pin, F.Cu at (327.1, 18.4)
- added REF**: Banana_Jack_1Pin, Connector:Banana_Jack_1Pin, F.Cu at (226.7, 18.7)
- added REF**: Banana_Jack_1Pin, Connector:Banana_Jack_1Pin, F.Cu at (470.5, 103.9)
- added REF**: Banana_Jack_1Pin, Connector:Banana_Jack_1Pin, F.Cu at (470.5, 66.2)
- added REF**: Banana_Jack_1Pin, Connector:Banana_Jack_1Pin, F.Cu at (467.3, 151.8)
- moved J1 28.3 mm to (168.9, 51.1)
- moved K79 23.2 mm to (212.7, 122.2)
- moved K80 15.3 mm to (231.7, 122.3)
- moved K83 5.20 mm to (330.8, 122.2)
- moved K84 5.20 mm to (349.8, 122.2)
- moved K85 5.20 mm to (368.9, 122.2)
- moved K65 5.20 mm to (349.8, 103.2)
- moved K27 5.15 mm to (335.5, 65.1)
- moved K28 5.15 mm to (364.1, 65.1)
- moved K56 4.77 mm to (126.8, 103.2)
- moved K70 4.77 mm to (34.1, 122.2)
- moved K72 4.77 mm to (79.3, 122.2)
- moved K73 4.77 mm to (98.4, 122.2)
- moved K74 4.77 mm to (117.4, 122.2)
- moved K75 4.77 mm to (136.5, 122.2)
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Routing:
- net /16: track 830.2 -> 530.0 mm, vias 1 -> 3
- net /22: track 496.9 -> 360.6 mm, vias 0 -> 1
- net /3: track 666.7 -> 542.6 mm, vias 1 -> 2
- net /21: track 502.7 -> 386.6 mm, vias 1 -> 3
- net /4: track 685.8 -> 575.8 mm, vias 0 -> 1
- net /1: track 392.4 -> 492.1 mm, vias 0 -> 3
- net /6: track 294.9 -> 202.4 mm, vias 0 -> 1
- net /24: track 521.3 -> 433.4 mm, vias 0 -> 1
- net /29: track 491.2 -> 411.8 mm, vias 0 -> 1
- net /26: track 361.3 -> 285.0 mm, vias 2 -> 1
- net /30: track 543.0 -> 473.5 mm, vias 0 -> 1
- net /18: track 605.4 -> 536.9 mm
- net /20: track 507.9 -> 457.7 mm, vias 1 -> 2
- net /23: track 383.2 -> 337.2 mm, vias 0 -> 1
- net /27: track 479.7 -> 436.7 mm, vias 0 -> 3
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Other:
- board size 460 x 149 mm -> 453 x 140 mm
- net class Default: clearance 0.2 -> 0.3; trace_width 0.25 -> 0.8; via_drill 0.4 -> 0.6
- rule trace_clearance: 0.2 -> 0.3
- rule trace_min: 0.9 -> 0.35
- rule via_min_drill: 0.3 -> 0.6
- rule via_min_size: 0.4 -> 0.8
- board text added: "Rev.2"
- board text added: "april 2019"
- board text removed: "Rev.1"
- board text removed: "march 2019"

Commit message: Submitted R2 to ourpcb
Routing:
- net /9: track 226.5 -> 223.5 mm, vias 2 -> 0
- net /31: track 271.9 -> 270.6 mm, vias 2 -> 0
Changed lines of the file:
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@@
     (thickness 2)
     (drawings 13)
-    (tracks 1280)
+    (tracks 1275)
     (zones 0)
     (modules 112)
@@
     (36 B.SilkS user hide)
     (37 F.SilkS user hide)
-    (38 B.Mask user hide)
-    (39 F.Mask user hide)
+    (38 B.Mask user)
+    (39 F.Mask user)
     (40 Dwgs.User user)
     (41 Cmts.User user hide)
@@
     (solder_mask_min_width 0.25)
     (aux_axis_origin 0 0)
-    (visible_elements FFFFE77F)
+    (visible_elements FFFFEF7F)
     (pcbplotparams
-      (layerselection 0x211c0_ffffffff)
+      (layerselection 0x011c0_ffffffff)
       (usegerberextensions false)
       (usegerberattributes false)
@@
   (segment (start 148.213138 51.19002) (end 150.650119 53.627001) (width 0.35) (layer F.Cu) (net 25))
   (segment (start 47.712982 51.19002) (end 148.213138 51.19002) (width 0.35) (layer F.Cu) (net 25))
-  (segment (start 442.838 136.272) (end 449.796 129.314) (width 0.35) (layer F.Cu) (net 26))
-  (segment (start 438.366 136.272) (end 442.838 136.272) (width 0.35) (layer F.Cu) (net 26))
   (segment (start 457.416 98.172) (end 438.366 98.172) (width 0.35) (layer F.Cu) (net 26))
   (segment (start 457.416 79.122) (end 438.366 79.122) (width 0.35) (layer F.Cu) (net 26))
@@
   (segment (start 153.330001 94.960001) (end 153.330001 71.970001) (width 0.35) (layer B.Cu) (net 26))
   (segment (start 153.83 95.46) (end 153.330001 94.960001) (width 0.35) (layer B.Cu) (net 26))
+  (segment (start 442.838 136.272) (end 449.796 129.314) (width 0.35) (layer B.Cu) (net 26))
+  (segment (start 438.366 136.272) (end 442.838 136.272) (width 0.35) (layer B.Cu) (net 26))
   (segment (start 57.767989 80.176493) (end 48.04 70.448504) (width 0.35) (layer B.Cu) (net 27))
   (segment (start 57.767989 113.039241) (end 57.767989 80.176493) (width 0.35) (layer B.Cu) (net 27))
@@
   (segment (start 76.857099 120.734903) (end 77.116001 120.476001) (width 0.35) (layer B.Cu) (net 28))
   (segment (start 69.42 136.218) (end 69.42 134.62701) (width 0.35) (layer B.Cu) (net 28))
-  (segment (start 51.894 109.5805) (end 51.7645 109.71) (width 0.35) (layer F.Cu) (net 29))
+  (segment (start 186.990762 49.89) (end 187.66 49.89) (width 0.35) (layer F.Cu) (net 29))
+  (segment (start 185.103751 48.002989) (end 186.990762 49.89) (width 0.35) (layer F.Cu) (net 29))
+  (segment (start 172.611493 48.002989) (end 185.103751 48.002989) (width 0.35) (layer F.Cu) (net 29))
+  (segment (start 171.961483 47.352979) (end 172.611493 48.002989) (width 0.35) (layer F.Cu) (net 29))
+  (segment (start 146.875326 44.03991) (end 148.784238 42.130998) (width 0.35) (layer F.Cu) (net 29))
+  (segment (start 166.188463 45.402951) (end 168.680721 45.402951) (width 0.35) (layer F.Cu) (net 29))
+  (segment (start 55.353003 43.060001) (end 56.982922 44.68992) (width 0.35) (layer F.Cu) (net 29))
+  (segment (start 150.85 42.802909) (end 162.007673 42.802909) (width 0.35) (layer F.Cu) (net 29))
+  (segment (start 165.525452 44.73994) (end 166.188463 45.402951) (width 0.35) (layer F.Cu) (net 29))
+  (segment (start 168.680721 45.402951) (end 170.630749 47.352979) (width 0.35) (layer F.Cu) (net 29))
+  (segment (start 104.65911 44.03991) (end 146.875326 44.03991) (width 0.35) (layer F.Cu) (net 29))
+  (segment (start 102.8181 43.1219) (end 103.7411 43.1219) (width 0.35) (layer F.Cu) (net 29))
+  (segment (start 170.630749 47.352979) (end 171.961483 47.352979) (width 0.35) (layer F.Cu) (net 29))
+  (segment (start 150.232002 42.130998) (end 150.85 42.748996) (width 0.35) (layer F.Cu) (net 29))
   (segment (start 51.894 108.278) (end 51.894 109.5805) (width 0.35) (layer F.Cu) (net 29))
-  (segment (start 51.7645 109.71) (end 20.54 109.71) (width 0.35) (layer F.Cu) (net 29))
-  (segment (start 20.54 109.71) (end 20.54 109.71) (width 0.35) (layer F.Cu) (net 29))
-  (via (at 20.54 109.71) (size 1) (drill 0.6) (layers F.Cu B.Cu) (net 29))
-  (segment (start 20.54 109.71) (end 20.54 43.56) (width 0.35) (layer B.Cu) (net 29))
-  (segment (start 20.54 43.56) (end 20.54 43.56) (width 0.35) (layer B.Cu) (net 29))
-  (via (at 20.54 43.56) (size 1) (drill 0.6) (layers F.Cu B.Cu) (net 29))
-  (segment (start 55.353003 43.060001) (end 21.039999 43.060001) (width 0.35) (layer F.Cu) (net 29))
-  (segment (start 56.982922 44.68992) (end 55.353003 43.060001) (width 0.35) (layer F.Cu) (net 29))
-  (segment (start 101.25008 44.68992) (end 56.982922 44.68992) (width 0.35) (layer F.Cu) (net 29))
-  (segment (start 104.65911 44.03991) (end 103.7411 43.1219) (width 0.35) (layer F.Cu) (net 29))
-  (segment (start 103.7411 43.1219) (end 102.8181 43.1219) (width 0.35) (layer F.Cu) (net 29))
-  (segment (start 148.784238 42.130998) (end 146.875326 44.03991) (width 0.35) (layer F.Cu) (net 29))
-  (segment (start 21.039999 43.060001) (end 20.54 43.56) (width 0.35) (layer F.Cu) (net 29))
-  (segment (start 150.85 42.748996) (end 150.232002 42.130998) (width 0.35) (layer F.Cu) (net 29))
-  (segment (start 185.103751 48.002989) (end 172.611493 48.002989) (width 0.35) (layer F.Cu) (net 29))
-  (segment (start 165.525452 44.73994) (end 163.944704 44.73994) (width 0.35) (layer F.Cu) (net 29))
-  (segment (start 146.875326 44.03991) (end 104.65911 44.03991) (width 0.35) (layer F.Cu) (net 29))
-  (segment (start 163.944704 44.73994) (end 162.007673 42.802909) (width 0.35) (layer F.Cu) (net 29))
-  (segment (start 162.007673 42.802909) (end 150.85 42.802909) (width 0.35) (layer F.Cu) (net 29))
-  (segment (start 187.66 49.89) (end 186.990762 49.89) (width 0.35) (layer F.Cu) (net 29))
-  (segment (start 168.680721 45.402951) (end 166.188463 45.402951) (width 0.35) (layer F.Cu) (net 29))
-  (segment (start 170.630749 47.352979) (end 168.680721 45.402951) (width 0.35) (layer F.Cu) (net 29))
-  (segment (start 166.188463 45.402951) (end 165.525452 44.73994) (width 0.35) (layer F.Cu) (net 29))
-  (segment (start 150.232002 42.130998) (end 148.784238 42.130998) (width 0.35) (layer F.Cu) (net 29))
-  (segment (start 172.611493 48.002989) (end 171.961483 47.352979) (width 0.35) (layer F.Cu) (net 29))
-  (segment (start 102.8181 43.1219) (end 101.25008 44.68992) (width 0.35) (layer F.Cu) (net 29))
-  (segment (start 150.85 42.802909) (end 150.85 42.748996) (width 0.35) (layer F.Cu) (net 29))
-  (segment (start 171.961483 47.352979) (end 170.630749 47.352979) (width 0.35) (layer F.Cu) (net 29))
-  (segment (start 186.990762 49.89) (end 185.103751 48.002989) (width 0.35) (layer F.Cu) (net 29))
-  (segment (start 49.354 108.278) (end 21.672 108.278) (width 0.35) (layer F.Cu) (net 30))
-  (segment (start 21.672 108.278) (end 21.672 108.278) (width 0.35) (layer F.Cu) (net 30))
-  (via (at 21.672 108.278) (size 1) (drill 0.6) (layers F.Cu B.Cu) (net 30))
-  (segment (start 21.672 108.278) (end 21.672 50.608) (width 0.35) (layer B.Cu) (net 30))
-  (segment (start 21.672 50.608) (end 21.672 50.608) (width 0.35) (layer B.Cu) (net 30))
-  (via (at 21.672 50.608) (size 1) (drill 0.6) (layers F.Cu B.Cu) (net 30))
+  (segment (start 148.784238 42.130998) (end 150.232002 42.130998) (width 0.35) (layer F.Cu) (net 29))
+  (segment (start 56.982922 44.68992) (end 101.25008 44.68992) (width 0.35) (layer F.Cu) (net 29))
+  (segment (start 24.89 110.36) (end 20.18 105.65) (width 0.35) (layer F.Cu) (net 29))
+  (segment (start 21.039999 43.060001) (end 55.353003 43.060001) (width 0.35) (layer F.Cu) (net 29))
+  (segment (start 103.7411 43.1219) (end 104.65911 44.03991) (width 0.35) (layer F.Cu) (net 29))
+  (segment (start 101.25008 44.68992) (end 102.8181 43.1219) (width 0.35) (layer F.Cu) (net 29))
+  (segment (start 20.18 43.92) (end 21.039999 43.060001) (width 0.35) (layer F.Cu) (net 29))
+  (segment (start 163.944704 44.73994) (end 165.525452 44.73994) (width 0.35) (layer F.Cu) (net 29))
+  (segment (start 150.85 42.748996) (end 150.85 42.802909) (width 0.35) (layer F.Cu) (net 29))
+  (segment (start 162.007673 42.802909) (end 163.944704 44.73994) (width 0.35) (layer F.Cu) (net 29))
+  (segment (start 51.1145 110.36) (end 24.89 110.36) (width 0.35) (layer F.Cu) (net 29))
+  (segment (start 51.894 109.5805) (end 51.1145 110.36) (width 0.35) (layer F.Cu) (net 29))
+  (segment (start 20.18 105.65) (end 20.18 43.92) (width 0.35) (layer F.Cu) (net 29))
   (segment (start 31.445001 48.914999) (end 29.752 50.608) (width 0.35) (layer F.Cu) (net 30))
   (segment (start 47.247006 49.23999) (end 33.322992 49.23999) (width 0.35) (layer F.Cu) (net 30))
@@
   (segment (start 50.326338 48.58998) (end 49.671356 47.934998) (width 0.35) (layer F.Cu) (net 30))
   (segment (start 33.322992 49.23999) (end 32.998001 48.914999) (width 0.35) (layer F.Cu) (net 30))
-  (segment (start 29.752 50.608) (end 21.672 50.608) (width 0.35) (layer F.Cu) (net 30))
   (segment (start 160.16 49.89) (end 158.272989 48.002989) (width 0.35) (layer F.Cu) (net 30))
   (segment (start 148.76002 48.58998) (end 50.326338 48.58998) (width 0.35) (layer F.Cu) (net 30))
   (segment (start 149.347011 48.002989) (end 148.76002 48.58998) (width 0.35) (layer F.Cu) (net 30))
+  (segment (start 23.748998 50.608) (end 21.48 52.876998) (width 0.35) (layer F.Cu) (net 30))
+  (segment (start 29.752 50.608) (end 23.748998 50.608) (width 0.35) (layer F.Cu) (net 30))
+  (segment (start 21.48 52.876998) (end 21.48 104.78) (width 0.35) (layer F.Cu) (net 30))
+  (segment (start 24.978 108.278) (end 49.354 108.278) (width 0.35) (layer F.Cu) (net 30))
+  (segment (start 21.48 104.78) (end 24.978 108.278) (width 0.35) (layer F.Cu) (net 30))
   (segment (start 452.666001 80.893999) (end 439.392903 67.620901) (width 0.35) (layer B.Cu) (net 32))
   (segment (start 452.666001 82.430001) (end 452.666001 80.893999) (width 0.35) (layer B.Cu) (net 32))
